Commit message: Added pybullet controller and bicopter_msgs.

File: bicopter_pybullet_controller/urdf/bicopter_urdf.urdf (robot description, URDF)
Before this commit: robot bicopter, 3 links, 2 joints
Links:
- link base: mass 0.3 -> 0.4; geometry collision mesh filename=/home/ebnerl/catkin_ws/src/bicopter/bicopter_pybullet_contr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 scale=0.001 0.001 0.001; visual mesh filename=/home/ebnerl/catkin_ws/src/bicopter/bicopter_pybullet_contr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 scale=0.001 0.001 0.001
- link propmount_left: geometry collision mesh filename=/home/ebnerl/catkin_ws/src/bicopter/bicopter_pybullet_contr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 scale=0.001 0.001 0.001; visual mesh filename=/home/ebnerl/catkin_ws/src/bicopter/bicopter_pybullet_contr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 scale=0.001 0.001 0.001
- link propmount_right: geometry collision mesh filename=/home/ebnerl/catkin_ws/src/bicopter/bicopter_pybullet_contr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 scale=0.001 0.001 0.001; visual mesh filename=/home/ebnerl/catkin_ws/src/bicopter/bicopter_pybullet_contr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 scale=0.001 0.001 0.001
