Commit message: Moved bicopter urdf to own package.

File: bicopter_model/urdf/bicopter_urdf.urdf (robot description, URDF)
Before this commit: robot bicopter, 3 links, 2 joints
Links:
- link base: geometry collision mesh filename=/home/ebnerl/catkin_ws/src/bicopter/bicopter_model/urdf/bic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 scale=0.001 0.001 0.001; visual mesh filename=/home/ebnerl/catkin_ws/src/bicopter/bicopter_model/urdf/bic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 scale=0.001 0.001 0.001
- link propmount_left: geometry collision mesh filename=/home/ebnerl/catkin_ws/src/bicopter/bicopter_model/urdf/bic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 scale=0.001 0.001 0.001; visual mesh filename=/home/ebnerl/catkin_ws/src/bicopter/bicopter_model/urdf/bic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 scale=0.001 0.001 0.001
- link propmount_right: geometry collision mesh filename=/home/ebnerl/catkin_ws/src/bicopter/bicopter_model/urdf/bic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 scale=0.001 0.001 0.001; visual mesh filename=/home/ebnerl/catkin_ws/src/bicopter/bicopter_model/urdf/bic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 scale=0.001 0.001 0.001

Commit message: Ported bicopter_model to ros2, fixed urdf test script

File: bicopter_model/urdf/bicopter_urdf.urdf (robot description, URDF)
Before this commit: robot bicopter, 3 links, 2 joints
Links:
- link base: geometry collision mesh filename=bicopter_base.stl scale=0.001 0.001 0.001; visual mesh filename=bicopter_base.stl scale=0.001 0.001 0.001
- link propmount_left: geometry collision mesh filename=bicopter_propmount.stl scale=0.001 0.001 0.001; visual mesh filename=bicopter_propmount.stl scale=0.001 0.001 0.001
- link propmount_right: geometry collision mesh filename=bicopter_propmount.stl scale=0.001 0.001 0.001; visual mesh filename=bicopter_propmount.stl scale=0.001 0.001 0.001
